Commit message: on passe à ycb:)

File: objets/7138_four/mobility.urdf (robot description, URDF)
Before this commit: robot partnet_19362facbca806df178e7d331e641179, 3 links, 2 joints
Links:
- link link_1: geometry collision mesh filename=textured_objs/new-0.obj; collision mesh filename=textured_objs/new-1.obj
